File: KiCad/wattson.kicad_sch (KiCad schematic)
At the start: 27 parts, among them Q2 NPN, SW1 Keypad 1, SW10 Plug, SW11 On/Off, SW2 Keypad 2, SW3 Keypad 3, SW4 Keypad 4, SW5 Keypad 5, SW6 Keypad 0, SW7 Keypad 6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

Commit message: move mcp interrupt pin, control vibration from DAC
Parts:
- added R8: 1k, symbol Device:R_US
- added U1: 24LC32, Adafruit HaD Proto HAT rev A:SOIC8_150MIL, symbol Adafruit HaD Proto HAT rev A-eagle-import:EEPROM_I2C_SOIC8_GENERIC
Connections:
- net +5V: no longer Q2.1 (C)
- net 3.3V: now also Q2.1 (C), U1.8 (VCC)
- net A0: now also Q2.2 (B), R8.2; no longer D1.3 (DIN)
- net GND: now also R8.1, U1.1 (A0), U1.2 (A1), U1.3 (A2), U1.4 (GND), U1.7 (WP)
- net SCL: now also D1.3 (DIN)
- net at R1.2, U2.13 (SDA): now also U1.5 (SDA)
- net at R2.2, U2.12 (SCK): now also U1.6 (SCL)
- net at U2.19 (INTB): no longer R7.2
- net at U2.20 (INTA): now also R7.2
- net at U2.3 (GPB2): no longer Q2.2 (B)

Commit message: Update schema, more docs
Parts:
- removed R6: 7,460, symbol Device:R_US
- SW1: value Keypad 1 -> BTN - Up
- SW2: value Keypad 2 -> BTN - Record
- SW3: value Keypad 3 -> BTN - Left
- SW4: value Keypad 4 -> BTN - Down
- SW5: value Keypad 5 -> BTN - Right
- SW6: value Keypad 0 -> BTN - Menu
- SW7: value Keypad 6 -> BTN - 1
- SW8: value Keypad 7 -> BTN - 2
Connections:
- net SCL is gone; now on net A1: D1.3 (DIN)
- net at U2.1 (GPB0): now also R4.2
- net at U2.2 (GPB1): now also R3.2
- net at U2.3 (GPB2): now also SW10.1
- net at U2.4 (GPB3): now also SW9.1
- net at U2.5 (GPB4): no longer SW9.1
- net at U2.6 (GPB5): no longer SW10.1
- net at U2.7 (GPB6): no longer R3.2
- net at U2.8 (GPB7): no longer R4.2
Other:
- company: (none) -> Zane Bauman
- title: (none) -> Wattson Heirloom
